File: hardware/DACs.kicad_sch (KiCad schematic)
At the start: 56 parts, among them J6 Conn_Coaxial, J7 Conn_Coaxial, J8 Conn_Coaxial, J9 Conn_Coaxial, U10 LTC2642, U11 LTC2642, U12 REF3525, U4 OPA2994IDGKR, U5 OPA2994IDGKR, U6 OPA2994IDGKR, U7 OPA2994IDGKR, U8 LTC2642, U9 LTC2642

Commit message: update footprints to meet min pad clearance of 0.2mm
Parts:
- U10, U11, U8, U9: footprint Package_SO:MSOP-10_3x3mm_P0.5mm -> kicad-lib:MSOP-10_3x3mm_P0.5mm_AnalogDevices
- U4, U5, U6, U7: footprint Package_SO:VSSOP-8_3x3mm_P0.65mm -> kicad-lib:VSSOP-8_3x3mm_P0.65mm_TexasInstruments
Changed lines of the file:
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@@
 			)
 		)
-		(property "Footprint" "Package_SO:VSSOP-8_3x3mm_P0.65mm"
+		(property "Footprint" "kicad-lib:VSSOP-8_3x3mm_P0.65mm_TexasInstruments"
 			(at 29.21 158.75 0)
 			(effects
@@
 			)
 		)
-		(property "Footprint" "Package_SO:VSSOP-8_3x3mm_P0.65mm"
+		(property "Footprint" "kicad-lib:VSSOP-8_3x3mm_P0.65mm_TexasInstruments"
 			(at 29.21 33.02 0)
 			(effects
@@
 			)
 		)
-		(property "Footprint" "Package_SO:VSSOP-8_3x3mm_P0.65mm"
+		(property "Footprint" "kicad-lib:VSSOP-8_3x3mm_P0.65mm_TexasInstruments"
 			(at 121.92 116.84 0)
 			(effects
@@
 			)
 		)
-		(property "Footprint" "Package_SO:VSSOP-8_3x3mm_P0.65mm"
+		(property "Footprint" "kicad-lib:VSSOP-8_3x3mm_P0.65mm_TexasInstruments"
 			(at 29.21 74.93 0)
 			(effects
@@
 			)
 		)
-		(property "Footprint" "Package_SO:VSSOP-8_3x3mm_P0.65mm"
+		(property "Footprint" "kicad-lib:VSSOP-8_3x3mm_P0.65mm_TexasInstruments"
 			(at 101.6 74.93 0)
 			(effects
@@
 			)
 		)
-		(property "Footprint" "Package_SO:VSSOP-8_3x3mm_P0.65mm"
+		(property "Footprint" "kicad-lib:VSSOP-8_3x3mm_P0.65mm_TexasInstruments"
 			(at 101.6 116.84 0)
 			(effects
@@
 			)
 		)
-		(property "Footprint" "Package_SO:MSOP-10_3x3mm_P0.5mm"
+		(property "Footprint" "kicad-lib:MSOP-10_3x3mm_P0.5mm_AnalogDevices"
 			(at 72.39 167.64 0)
 			(effects
@@
 			)
 		)
-		(property "Footprint" "Package_SO:VSSOP-8_3x3mm_P0.65mm"
+		(property "Footprint" "kicad-lib:VSSOP-8_3x3mm_P0.65mm_TexasInstruments"
 			(at 101.6 158.75 0)
 			(effects
@@
 			)
 		)
-		(property "Footprint" "Package_SO:VSSOP-8_3x3mm_P0.65mm"
+		(property "Footprint" "kicad-lib:VSSOP-8_3x3mm_P0.65mm_TexasInstruments"
 			(at 29.21 116.84 0)
 			(effects
@@
 			)
 		)
-		(property "Footprint" "Package_SO:VSSOP-8_3x3mm_P0.65mm"
+		(property "Footprint" "kicad-lib:VSSOP-8_3x3mm_P0.65mm_TexasInstruments"
 			(at 121.92 74.93 0)
 			(effects
@@
 			)
 		)
-		(property "Footprint" "Package_SO:VSSOP-8_3x3mm_P0.65mm"
+		(property "Footprint" "kicad-lib:VSSOP-8_3x3mm_P0.65mm_TexasInstruments"
 			(at 121.92 158.75 0)
 			(effects
@@
 			)
 		)
-		(property "Footprint" "Package_SO:MSOP-10_3x3mm_P0.5mm"
+		(property "Footprint" "kicad-lib:MSOP-10_3x3mm_P0.5mm_AnalogDevices"
 			(at 72.39 125.73 0)
 			(effects
@@
 			)
 		)
-		(property "Footprint" "Package_SO:VSSOP-8_3x3mm_P0.65mm"
+		(property "Footprint" "kicad-lib:VSSOP-8_3x3mm_P0.65mm_TexasInstruments"
 			(at 101.6 33.02 0)
 			(effects
@@
 			)
 		)
-		(property "Footprint" "Package_SO:VSSOP-8_3x3mm_P0.65mm"
+		(property "Footprint" "kicad-lib:VSSOP-8_3x3mm_P0.65mm_TexasInstruments"
 			(at 121.92 33.02 0)
 			(effects
@@
 			)
 		)
-		(property "Footprint" "Package_SO:MSOP-10_3x3mm_P0.5mm"
+		(property "Footprint" "kicad-lib:MSOP-10_3x3mm_P0.5mm_AnalogDevices"
 			(at 72.39 83.82 0)
 			(effects
@@
 			)
 		)
-		(property "Footprint" "Package_SO:MSOP-10_3x3mm_P0.5mm"
+		(property "Footprint" "kicad-lib:MSOP-10_3x3mm_P0.5mm_AnalogDevices"
 			(at 72.39 41.91 0)
 			(effects

Commit message: update 1K, 31K6, 10K resistors to 0.1%
Parts:
- R1, R19, R22, R23, R24, R25, R26, R27, R28, R29, R30, R4: Link https://www.digikey.com/en/products/detail/samsung-electro-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 -> https://www.digikey.com/en/products/detail/yageo/RT0402BRD0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; Manufacturer Samsung Electro-Mechanics -> YAGEO; Manufacturer Number RC1005F103CS -> RT0402BRD0710KL; Tolerance (none) -> 0.1%

Commit message: swap BNC connectors to taller versions
Parts:
- J6, J7, J8, J9: footprint kicad-lib:BNC_TEConnectivity_CONBNC001_Vertical -> kicad-lib:BNC_AmphenolRF_031-5329-52RFX_Vertical; Link https://www.digikey.com/en/products/detail/te-connectivity-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 -> https://www.digikey.com/en/products/detail/amphenol-rf/031-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; Manufacturer TE Connectivity Linx -> Amphenol RF
Changed lines of the file:
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@@
 			)
 		)
-		(property "Footprint" "kicad-lib:BNC_TEConnectivity_CONBNC001_Vertical"
+		(property "Footprint" "kicad-lib:BNC_AmphenolRF_031-5329-52RFX_Vertical"
 			(at 158.75 77.47 0)
 			(effects
@@
 			)
 		)
-		(property "Datasheet" "https://www.te.com/commerce/DocumentDelivery/DDEController?Action=srchrtrv&DocNm=CONBNC001&DocType=Data+Sheet&DocLang=English&DocFormat=pdf&PartCntxt=CONBNC001"
+		(property "Datasheet" "https://www.amphenolrf.com/en-us/assets/file/4065788070/"
 			(at 158.75 77.47 0)
 			(effects
@@
 			)
 		)
-		(property "Link" "https://www.digikey.com/en/products/detail/te-connectivity-linx/CONBNC001/16013844"
+		(property "Link" "https://www.digikey.com/en/products/detail/amphenol-rf/031-5329-52RFX/2041814"
 			(at 158.75 77.47 0)
 			(effects
@@
 			)
 		)
-		(property "Manufacturer" "TE Connectivity Linx"
+		(property "Manufacturer" "Amphenol RF"
 			(at 158.75 77.47 0)
 			(effects
@@
 			)
 		)
-		(property "Footprint" "kicad-lib:BNC_TEConnectivity_CONBNC001_Vertical"
+		(property "Footprint" "kicad-lib:BNC_AmphenolRF_031-5329-52RFX_Vertical"
 			(at 158.75 161.29 0)
 			(effects
@@
 			)
 		)
-		(property "Datasheet" "https://www.te.com/commerce/DocumentDelivery/DDEController?Action=srchrtrv&DocNm=CONBNC001&DocType=Data+Sheet&DocLang=English&DocFormat=pdf&PartCntxt=CONBNC001"
+		(property "Datasheet" "https://www.amphenolrf.com/en-us/assets/file/4065788070/"
 			(at 158.75 161.29 0)
 			(effects
@@
 			)
 		)
-		(property "Link" "https://www.digikey.com/en/products/detail/te-connectivity-linx/CONBNC001/16013844"
+		(property "Link" "https://www.digikey.com/en/products/detail/amphenol-rf/031-5329-52RFX/2041814"
 			(at 158.75 161.29 0)
 			(effects
@@
 			)
 		)
-		(property "Manufacturer" "TE Connectivity Linx"
+		(property "Manufacturer" "Amphenol RF"
 			(at 158.75 161.29 0)
 			(effects
@@
 			)
 		)
-		(property "Footprint" "kicad-lib:BNC_TEConnectivity_CONBNC001_Vertical"
+		(property "Footprint" "kicad-lib:BNC_AmphenolRF_031-5329-52RFX_Vertical"
 			(at 158.75 119.38 0)
 			(effects
@@
 			)
 		)
-		(property "Datasheet" "https://www.te.com/commerce/DocumentDelivery/DDEController?Action=srchrtrv&DocNm=CONBNC001&DocType=Data+Sheet&DocLang=English&DocFormat=pdf&PartCntxt=CONBNC001"
+		(property "Datasheet" "https://www.amphenolrf.com/en-us/assets/file/4065788070/"
 			(at 158.75 119.38 0)
 			(effects
@@
 			)
 		)
-		(property "Link" "https://www.digikey.com/en/products/detail/te-connectivity-linx/CONBNC001/16013844"
+		(property "Link" "https://www.digikey.com/en/products/detail/amphenol-rf/031-5329-52RFX/2041814"
 			(at 158.75 119.38 0)
 			(effects
@@
 			)
 		)
-		(property "Manufacturer" "TE Connectivity Linx"
+		(property "Manufacturer" "Amphenol RF"
 			(at 158.75 119.38 0)
 			(effects
@@
 			)
 		)
-		(property "Footprint" "kicad-lib:BNC_TEConnectivity_CONBNC001_Vertical"
+		(property "Footprint" "kicad-lib:BNC_AmphenolRF_031-5329-52RFX_Vertical"
 			(at 158.75 35.56 0)
 			(effects
@@
 			)
 		)
-		(property "Datasheet" "https://www.te.com/commerce/DocumentDelivery/DDEController?Action=srchrtrv&DocNm=CONBNC001&DocType=Data+Sheet&DocLang=English&DocFormat=pdf&PartCntxt=CONBNC001"
+		(property "Datasheet" "https://www.amphenolrf.com/en-us/assets/file/4065788070/"
 			(at 158.75 35.56 0)
 			(effects
@@
 			)
 		)
-		(property "Link" "https://www.digikey.com/en/products/detail/te-connectivity-linx/CONBNC001/16013844"
+		(property "Link" "https://www.digikey.com/en/products/detail/amphenol-rf/031-5329-52RFX/2041814"
 			(at 158.75 35.56 0)
 			(effects
@@
 			)
 		)
-		(property "Manufacturer" "TE Connectivity Linx"
+		(property "Manufacturer" "Amphenol RF"
 			(at 158.75 35.56 0)
 			(effects
