File: hardware/DACs.kicad_sch (KiCad schematic)
At the start: 56 parts, among them J6 Conn_Coaxial, J7 Conn_Coaxial, J8 Conn_Coaxial, J9 Conn_Coaxial, U10 LTC2642, U11 LTC2642, U12 REF3525, U4 OPA2994IDGKR, U5 OPA2994IDGKR, U6 OPA2994IDGKR, U7 OPA2994IDGKR, U8 LTC2642, U9 LTC2642

Commit message: Dev -> Main (#85)
* draft dma double buffer

* cleanup dma double buffer draft

* draft double buffer

* redraft dma double buffer

* get ping pong re-triggering

* draft double buffer with example

* get buffer -> dma-> pio working

* draft sd card to dac for 1 channel

* get single chan sd-to-dac working

* redraft file iteration with linked list

* get large transfers working

* draft multichannel sd -> dma -> dac

* cleanup 4 channel sd to dac example

* update pio ltc264x lib

* add pause/resume with test

* valdiate abort_transfer fn

* draft MultiFilePlayer

* draft multi file player class

* add/test is_aborted and reset_transfer_config after abort

* update abort example

* draft test for multi file player

* cleanup multi_file_player.h

* cleanup double buffer comments

* get multi file player example working

* remove hardcoding in abort func

* draft harp interface

* add missing register

* Update README.md

* Update README.md

* Update README.md

* Update README.md

* Update README.md

* Update README.md

* Update README.md

* add placeholder graphic

* Update README.md

* Update README.md

* fix sd switch card profiling test pinout

* Update README.md

* Update README.md

* Update README.md

* Update README.md

* Update README.md

* Update README.md

* Update README.md

* add placeholder graphic

* Update README.md

* Update README.md

* draft device.yml

* draft is_ready and start-from-harp

* draft one-shot analog output

* draft external hw trigger logic

* update waveform default settings

* cleanup draft; fix compiler errors

* generate bitmasks from template at compile time

* draft pyharp tests

* add sw trigger pyharp test

* draft optional end-of-transfer to trigger IRQ & send harp EVENT

* cleanup isr callback; enable override

* update multifileplayer pinout

* update pause_and_resume test pinout

* update abort test pinout

* update read_sd_card test

* update buf-to-dac pinout

* update multifileplayer to zero output and record timestamp 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
Parts:
- J6, J7, J8, J9: footprint kicad-lib:BNC_TEConnectivity_CONBNC001_Vertical -> kicad-lib:BNC_AmphenolRF_031-5329-52RFX_Vertical; Link https://www.digikey.com/en/products/detail/te-connectivity-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 -> https://www.digikey.com/en/products/detail/amphenol-rf/031-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; Manufacturer TE Connectivity Linx -> Amphenol RF
- R1, R19, R22, R23, R24, R25, R26, R27, R28, R29, R30, R4: Link https://www.digikey.com/en/products/detail/samsung-electro-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 -> https://www.digikey.com/en/products/detail/yageo/RT0402BRD0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; Manufacturer Samsung Electro-Mechanics -> YAGEO; Manufacturer Number RC1005F103CS -> RT0402BRD0710KL; Tolerance (none) -> 0.1%
- U4, U5, U6, U7: value OPA2994IDGKR -> OPA2810IDGKT; Link (none) -> https://www.digikey.com/en/products/detail/texas-instrument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; Manufacturer Number OPA2994IDGKR -> OPA2810IDGKT
