File: hardware/SC_Detection.kicad_sch (KiCad schematic)
At the start: 58 parts, among them U13 LMV393IDGKR, U14 LMV393IDGKR, U15 LMV393IDGKR, U16 LMV393IDGKR, U17 INA630, U18 INA630, U19 INA630, U20 INA630, U21 REF2033

Commit message: update 1K, 31K6, 10K resistors to 0.1%
Parts:
- R39, R42, R43, R46, R47, R50, R51, R54: Link (none) -> https://www.digikey.com/en/products/detail/yageo/RT0402BRD0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; Manufacturer Number RC0402FR-0731K6L -> RT0402BRD0731K6L
- R40, R41, R44, R45, R48, R49, R52, R53, R80, R82, R84, R86: Link https://www.digikey.com/en/products/detail/panasonic-electr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 -> https://www.digikey.com/en/products/detail/yageo/RT0402BRE0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; Manufacturer Panasonic Electronic Components -> YAGEO; Manufacturer Number ERJ-2RKF1001X -> RT0402BRE071KL; Tolerance (none) -> 0.1%
- R55, R56, R57, R58: Link https://www.digikey.com/en/products/detail/samsung-electro-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 -> https://www.digikey.com/en/products/detail/yageo/RT0402BRD0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; Manufacturer Samsung Electro-Mechanics -> YAGEO; Manufacturer Number RC1005F103CS -> RT0402BRD0710KL; Tolerance (none) -> 0.1%
