File: hardware/SC_Detection.kicad_sch (KiCad schematic)
At the start: 58 parts, among them U13 LMV393IDGKR, U14 LMV393IDGKR, U15 LMV393IDGKR, U16 LMV393IDGKR, U17 INA630, U18 INA630, U19 INA630, U20 INA630, U21 REF2033

Commit message: update schematic component metadata
Parts:
- U17, U18, U19, U20: Manufacturer Number (none) -> INA630DDFR
Changed lines of the file:
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@@
 			)
 		)
+		(property "Manufacturer Number" "INA630DDFR"
+			(at 90.17 88.9 0)
+			(effects
+				(font
+					(size 1.27 1.27)
+				)
+				(hide yes)
+			)
+		)
 		(pin "1"
 		)
@@
 			)
 		)
+		(property "Manufacturer Number" "INA630DDFR"
+			(at 90.17 130.81 0)
+			(effects
+				(font
+					(size 1.27 1.27)
+				)
+				(hide yes)
+			)
+		)
 		(pin "1"
 		)
@@
 			)
 		)
+		(property "Manufacturer Number" "INA630DDFR"
+			(at 90.17 46.99 0)
+			(effects
+				(font
+					(size 1.27 1.27)
+				)
+				(hide yes)
+			)
+		)
 		(pin "1"
 		)
@@
 			(effects
 				(font
+					(size 1.27 1.27)
+				)
+				(hide yes)
+			)
+		)
+		(property "Manufacturer Number" "INA630DDFR"
+			(at 90.17 172.72 0)
+			(effects
+				(font
