File: hardware/Input.kicad_sch (KiCad schematic)
At the start: 19 parts, among them J10 Conn_Coaxial, J11 Conn_Coaxial, J12 Conn_Coaxial, J13 Conn_Coaxial, U22 SN74LVC2T45DCTR, U23 SN74LVC2T45DCTR

Commit message: update schematic component metadata
Parts:
- D11, D12, D13, D14: Alternate (none) -> VBUS05N1-HD1HG3-08
Changed lines of the file:
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@@
 			)
 		)
+		(property "Alternate" "VBUS05N1-HD1HG3-08"
+			(at 124.46 143.51 90)
+			(effects
+				(font
+					(size 1.27 1.27)
+				)
+				(hide yes)
+			)
+		)
 		(pin "1"
 		)
@@
 			)
 		)
+		(property "Alternate" "VBUS05N1-HD1HG3-08"
+			(at 124.46 85.09 90)
+			(effects
+				(font
+					(size 1.27 1.27)
+				)
+				(hide yes)
+			)
+		)
 		(pin "1"
 		)
@@
 			)
 		)
+		(property "Alternate" "VBUS05N1-HD1HG3-08"
+			(at 124.46 121.92 90)
+			(effects
+				(font
+					(size 1.27 1.27)
+				)
+				(hide yes)
+			)
+		)
 		(pin "1"
 		)
@@
 			(at 124.46 64.77 90)
 			(effects
+				(font
+					(size 1.27 1.27)
+				)
+				(hide yes)
+			)
+		)
+		(property "Alternate" "VBUS05N1-HD1HG3-08"
+			(at 124.46 64.77 90)
+			(effects
